File: cockpit/panels/MCP/hardware/electronics/mcpElectronics/altitude.kicad_sch (KiCad schematic)
At the start: 27 parts

Commit message: update
Parts:
- removed C? (x5): 100n, symbol Device:C
- removed R? (x5): 1k, symbol Device:R
- removed U? (x5): TLC5916IDR, TLC5916IDR:SOIC127P600X175-16N, symbol TLC5916IDR:TLC5916IDR
- removed U? (x5): WHITE_7_SEGMENT_LED, Display_7Segment:Sx39-1xxxxx, symbol Display_Character:SA39-11EWA
- added C4 (x5): 100n, Capacitor_SMD:C_0402_1005Metric, symbol Device:C
- added J18 (x5): WHITE_7_SEGMENT_LED, Connector_PinHeader_2.54mm:PinHeader_1x09_P2.54mm_Vertical, symbol Connector:Conn_01x09_Pin
- added R139 (x2): 4k7, Resistor_SMD:R_0402_1005Metric, symbol Device:R
- C59, C60: renamed from C?; footprint (none) -> Capacitor_SMD:C_0402_1005Metric
- R122, R123: renamed from R?; footprint (none) -> Resistor_SMD:R_0402_1005Metric
- SW17: renamed from SW?; footprint (none) -> Rotary_Encoder:RotaryEncoder_Bourns_Vertical_PEC12R-3x17F-Nxxxx
- SW18, SW19: renamed from SW?; footprint (none) -> Button_Switch_THT:SW_PUSH_6mm_H5mm
Connections:
- net +3V3: now also R139.1, R139.1
- net ALTITUDE_DEC: now also R139.2
- net ALTITUDE_INC: now also R139.2
- net Earth: now also C4.2, C4.2, C4.2, C4.2, C4.2
- new net LEDS_ANODE_12: C4.1, J18.8 (Pin_8), J18.9 (Pin_9)
- new net LEDS_ANODE_13: C4.1, J18.8 (Pin_8), J18.9 (Pin_9)
- new net LEDS_ANODE_14: C4.1, J18.8 (Pin_8), J18.9 (Pin_9)
- new net LEDS_ANODE_15: C4.1, J18.8 (Pin_8), J18.9 (Pin_9)
- new net LEDS_ANODE_16: C4.1, J18.8 (Pin_8), J18.9 (Pin_9)
- new net LEDS_SEGMENTS_ROW_A: J18.1 (Pin_1), J18.1 (Pin_1), J18.1 (Pin_1), J18.1 (Pin_1), J18.1 (Pin_1)
- new net LEDS_SEGMENTS_ROW_B: J18.2 (Pin_2), J18.2 (Pin_2), J18.2 (Pin_2), J18.2 (Pin_2), J18.2 (Pin_2)
- new net LEDS_SEGMENTS_ROW_C: J18.3 (Pin_3), J18.3 (Pin_3), J18.3 (Pin_3), J18.3 (Pin_3), J18.3 (Pin_3)
- new net LEDS_SEGMENTS_ROW_D: J18.4 (Pin_4), J18.4 (Pin_4), J18.4 (Pin_4), J18.4 (Pin_4), J18.4 (Pin_4)
- new net LEDS_SEGMENTS_ROW_E: J18.5 (Pin_5), J18.5 (Pin_5), J18.5 (Pin_5), J18.5 (Pin_5), J18.5 (Pin_5)
- new net LEDS_SEGMENTS_ROW_F: J18.6 (Pin_6), J18.6 (Pin_6), J18.6 (Pin_6), J18.6 (Pin_6), J18.6 (Pin_6)
- new net LEDS_SEGMENTS_ROW_G: J18.7 (Pin_7), J18.7 (Pin_7), J18.7 (Pin_7), J18.7 (Pin_7), J18.7 (Pin_7)
- no-connect marks 11 -> 0
