File: cockpit/panels/MCP/hardware/electronics/mcpElectronics/ap.kicad_sch (KiCad schematic)
At the start: 18 parts

Commit message: update schematic
Parts:
- added J?: A/P_DISENGAGE_BUTTON, symbol Connector:Conn_01x02_Male
- added R?: 10k, symbol Device:R
Connections:
- net +3V3: now also R?.1
- net Earth: now also J?.2 (Pin_2)
- new net A/P_DISENGAGE: J?.1 (Pin_1), R?.2
Changed lines of the file:
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@@
   (junction (at 173.99 97.79) (diameter 0) (color 0 0 0 0)
   )
+  (junction (at 243.84 76.2) (diameter 0) (color 0 0 0 0)
+  )
   (junction (at 86.36 101.6) (diameter 0) (color 0 0 0 0)
   )
@@
     (stroke (width 0) (type default) (color 0 0 0 0))
   )
+  (wire (pts (xy 234.95 73.66) (xy 234.95 76.2))
+    (stroke (width 0) (type default) (color 0 0 0 0))
+  )
   (wire (pts (xy 96.52 69.85) (xy 96.52 63.5))
     (stroke (width 0) (type default) (color 0 0 0 0))
@@
     (stroke (width 0) (type default) (color 0 0 0 0))
   )
+  (wire (pts (xy 243.84 76.2) (xy 248.92 76.2))
+    (stroke (width 0) (type default) (color 0 0 0 0))
+  )
   (wire (pts (xy 45.72 95.25) (xy 49.53 95.25))
     (stroke (width 0) (type default) (color 0 0 0 0))
@@
     (stroke (width 0) (type default) (color 0 0 0 0))
   )
+  (wire (pts (xy 237.49 73.66) (xy 237.49 76.2))
+    (stroke (width 0) (type default) (color 0 0 0 0))
+  )
   (wire (pts (xy 49.53 63.5) (xy 55.88 63.5))
     (stroke (width 0) (type default) (color 0 0 0 0))
   )
+  (wire (pts (xy 237.49 76.2) (xy 243.84 76.2))
+    (stroke (width 0) (type default) (color 0 0 0 0))
+  )
   (wire (pts (xy 35.56 69.85) (xy 36.83 69.85))
     (stroke (width 0) (type default) (color 0 0 0 0))
@@
     (stroke (width 0) (type default) (color 0 0 0 0))
   )
+  (wire (pts (xy 243.84 72.39) (xy 243.84 76.2))
+    (stroke (width 0) (type default) (color 0 0 0 0))
+  )
   (wire (pts (xy 45.72 63.5) (xy 49.53 63.5))
     (stroke (width 0) (type default) (color 0 0 0 0))
@@
     (effects (font (size 1.27 1.27)) (justify left))
     (property "Intersheet References" "${INTERSHEET_REFS}" (id 0) (at 70.4488 63.4206 0)
+      (effects (font (size 1.27 1.27)) (justify left) hide)
+    )
+  )
+  (global_label "A{slash}P_DISENGAGE" (shape output) (at 248.92 76.2 0) (fields_autoplaced)
+    (effects (font (size 1.27 1.27)) (justify left))
+    (property "Intersheet References" "${INTERSHEET_REFS}" (id 0) (at 266.3312 76.1206 0)
       (effects (font (size 1.27 1.27)) (justify left) hide)
     )
@@
     (pin "2")
   )
+  (symbol (lib_id "Connector:Conn_01x02_Male") (at 237.49 68.58 270) (unit 1)
+    (in_bom yes) (on_board yes)
+    (property "Reference" "J?" (id 0) (at 228.6 69.85 90)
+      (effects (font (size 1.27 1.27)) (justify left))
+    )
+    (property "Value" "A/P_DISENGAGE_BUTTON" (id 1) (at 208.28 72.39 90)
+      (effects (font (size 1.27 1.27)) (justify left))
+    )
+    (property "Footprint" "" (id 2) (at 237.49 68.58 0)
+      (effects (font (size 1.27 1.27)) hide)
+    )
+    (property "Datasheet" "~" (id 3) (at 237.49 68.58 0)
+      (effects (font (size 1.27 1.27)) hide)
+    )
+    (pin "1")
+    (pin "2")
+  )
   (symbol (lib_id "power:+3V3") (at 100.33 87.63 0) (unit 1)
     (in_bom yes) (on_board yes) (fields_autoplaced)
@@
     (pin "2")
   )
+  (symbol (lib_id "Device:R") (at 243.84 68.58 0) (unit 1)
+    (in_bom yes) (on_board yes)
+    (property "Reference" "R?" (id 0) (at 246.38 67.31 0)
+      (effects (font (size 1.27 1.27)) (justify left))
+    )
+    (property "Value" "10k" (id 1) (at 246.38 69.85 0)
+      (effects (font (size 1.27 1.27)) (justify left))
+    )
+    (property "Footprint" "" (id 2) (at 242.062 68.58 90)
+      (effects (font (size 1.27 1.27)) hide)
+    )
+    (property "Datasheet" "~" (id 3) (at 243.84 68.58 0)
+      (effects (font (size 1.27 1.27)) hide)
+    )
+    (pin "1")
+    (pin "2")
+  )
   (symbol (lib_id "Device:R") (at 49.53 59.69 0) (unit 1)
     (in_bom yes) (on_board yes) (fields_autoplaced)
@@
     (pin "1")
   )
+  (symbol (lib_id "power:+3V3") (at 243.84 64.77 0) (unit 1)
+    (in_bom yes) (on_board yes) (fields_autoplaced)
+    (property "Reference" "#PWR?" (id 0) (at 243.84 68.58 0)
+      (effects (font (size 1.27 1.27)) hide)
+    )
+    (property "Value" "+3V3" (id 1) (at 243.84 59.69 0))
+    (property "Footprint" "" (id 2) (at 243.84 64.77 0)
+      (effects (font (size 1.27 1.27)) hide)
+    )
+    (property "Datasheet" "" (id 3) (at 243.84 64.77 0)
+      (effects (font (size 1.27 1.27)) hide)
+    )
+    (pin "1")
+  )
   (symbol (lib_id "power:Earth") (at 157.48 96.52 0) (unit 1)
     (in_bom yes) (on_board yes) (fields_autoplaced)
@@
     (pin "2")
   )
+  (symbol (lib_id "power:Earth") (at 234.95 76.2 0) (unit 1)
+    (in_bom yes) (on_board yes) (fields_autoplaced)
+    (property "Reference" "#PWR?" (id 0) (at 234.95 82.55 0)
+      (effects (font (size 1.27 1.27)) hide)
+    )
+    (property "Value" "Earth" (id 1) (at 234.95 80.01 0)
+      (effects (font (size 1.27 1.27)) hide)
+    )
+    (property "Footprint" "" (id 2) (at 234.95 76.2 0)
+      (effects (font (size 1.27 1.27)) hide)
+    )
+    (property "Datasheet" "~" (id 3) (at 234.95 76.2 0)
+      (effects (font (size 1.27 1.27)) hide)
+    )
+    (pin "1")
+  )
   (symbol (lib_id "Switch:SW_SPDT") (at 166.37 64.77 0) (unit 1)

Commit message: update
Parts:
- removed R? (x2): 10k, symbol Device:R
- C61, C62, C63, C64: renamed from C?; footprint (none) -> Capacitor_SMD:C_0402_1005Metric
- J15: renamed from J?; footprint (none) -> Connector_PinHeader_2.54mm:PinHeader_1x02_P2.54mm_Vertical
- R124, R125, R126, R127, R128, R129, R130: renamed from R?; footprint (none) -> Resistor_SMD:R_0402_1005Metric
- SW21, SW22, SW23, SW24: renamed from SW?; footprint (none) -> Button_Switch_THT:SW_PUSH_6mm_H5mm
- SW25, SW26: renamed from SW?; footprint (none) -> Connector_PinHeader_2.54mm:PinHeader_1x02_P2.54mm_Vertical
Connections:
- net F/D_A_OFF: no longer names the net of SW25.3 (C)
- net F/D_B_OFF: no longer names the net of SW26.3 (C)
- no-connect marks 0 -> 2
