File: cockpit/panels/MCP/hardware/electronics/mcpElectronics/general.kicad_sch (KiCad schematic)
At the start: 1 part

Commit message: update
Parts:
- removed U?: MCP4018-xxxxLT, Package_TO_SOT_SMD:SOT-363_SC-70-6, symbol Potentiometer_Digital:MCP4018-xxxxLT
- added C1, C66: 1u, Capacitor_SMD:C_0402_1005Metric, symbol Device:C
- added C2, C67: 10u, Capacitor_SMD:C_0603_1608Metric, symbol Device:C
- added D1, D10, D11, D12, D13, D14, D2, D3, D4, D5, D6, D7, D8, D9: LED, Connector_PinHeader_2.54mm:PinHeader_1x02_P2.54mm_Vertical, symbol Device:LED
- added H1, H2, H3, H4: MountingHole_Pad, MountingHole:MountingHole_4.3mm_M4_ISO7380_Pad, symbol Mechanical:MountingHole_Pad
- added J10: BACKLIGHT_BULB_6, Connector_PinHeader_2.54mm:PinHeader_1x02_P2.54mm_Vertical, symbol Connector_Generic:Conn_01x02
- added J11: BACKLIGHT_BULB_7, Connector_PinHeader_2.54mm:PinHeader_1x02_P2.54mm_Vertical, symbol Connector_Generic:Conn_01x02
- added J12: BACKLIGHT_BULB_8, Connector_PinHeader_2.54mm:PinHeader_1x02_P2.54mm_Vertical, symbol Connector_Generic:Conn_01x02
- added J13: BACKLIGHT_BULB_9, Connector_PinHeader_2.54mm:PinHeader_1x02_P2.54mm_Vertical, symbol Connector_Generic:Conn_01x02
- added J17: ST-Link_Conn, Connector_PinHeader_2.54mm:PinHeader_1x04_P2.54mm_Vertical, symbol Connector:Conn_01x04_Pin
- added J4: BACKLIGHT_BULB_0, Connector_PinHeader_2.54mm:PinHeader_1x02_P2.54mm_Vertical, symbol Connector_Generic:Conn_01x02
- added J5: BACKLIGHT_BULB_1, Connector_PinHeader_2.54mm:PinHeader_1x02_P2.54mm_Vertical, symbol Connector_Generic:Conn_01x02
- added J6: BACKLIGHT_BULB_2, Connector_PinHeader_2.54mm:PinHeader_1x02_P2.54mm_Vertical, symbol Connector_Generic:Conn_01x02
- added J7: BACKLIGHT_BULB_3, Connector_PinHeader_2.54mm:PinHeader_1x02_P2.54mm_Vertical, symbol Connector_Generic:Conn_01x02
- added J8: BACKLIGHT_BULB_4, Connector_PinHeader_2.54mm:PinHeader_1x02_P2.54mm_Vertical, symbol Connector_Generic:Conn_01x02
- added J9: BACKLIGHT_BULB_5, Connector_PinHeader_2.54mm:PinHeader_1x02_P2.54mm_Vertical, symbol Connector_Generic:Conn_01x02
- added Q1, Q10, Q11, Q12, Q13, Q14, Q15, Q16, Q17, Q18, Q19, Q2, Q20, Q21, Q22, Q23, Q24, Q3, Q4, Q5, Q6, Q7, Q8, Q9: C945, Package_TO_SOT_THT:TO-92_Inline, symbol Simulation_SPICE:NPN
- added Q32 (x9): S8050, Package_TO_SOT_THT:TO-92_Inline, symbol Transistor_BJT:S8050
- added R1, R10, R11, R12, R13, R14, R15, R16, R17, R18, R19, R2, R20, R21, R22, R23, R24, R25, R26, R27, R28, R29, R3, R30, R31, R32, R33, R34, R35, R36, R37, R38, R39, R4, R40, R41, R42, R43, R44, R45, R46, R47, R48, R49, R5, R50, R51, R52, R53, R54, R55, R57, R58, R6, R7, R8, R9: 560R, Resistor_SMD:R_0402_1005Metric, symbol Device:R
- added R107: 0R, Resistor_THT:R_Axial_DIN0207_L6.3mm_D2.5mm_P10.16mm_Horizontal, symbol Device:R
- added R59, R60, R61, R62, R63, R64, R65, R66, R67, R68, R69, R70, R71, R72: 330R, Resistor_SMD:R_0402_1005Metric, symbol Device:R
Connections:
- net Earth: now also C1.2, C2.2, C66.2, C67.2, H1.1, H2.1, H3.1, H4.1, J17.1 (Pin_1), Q32.1 (E), Q32.1 (E), Q32.1 (E), Q32.1 (E), Q32.1 (E), Q32.1 (E), Q32.1 (E), Q32.1 (E), Q32.1 (E)
- new net: Q17.1 (C), R17.1
- new net: Q17.2 (B), R48.2
- new net: J10.1 (Pin_1), J11.1 (Pin_1), J12.1 (Pin_1), J13.1 (Pin_1), J4.1 (Pin_1), J5.1 (Pin_1), J6.1 (Pin_1), J7.1 (Pin_1), J8.1 (Pin_1), J9.1 (Pin_1), Q32.3 (C)
- new net: J10.2 (Pin_2), J11.2 (Pin_2), J12.2 (Pin_2), J13.2 (Pin_2), J4.2 (Pin_2), J5.2 (Pin_2), J6.2 (Pin_2), J7.2 (Pin_2), J8.2 (Pin_2), J9.2 (Pin_2), R107.1
- new net: Q16.2 (B), R47.2
- new net: Q16.1 (C), R16.1
- new net: Q3.2 (B), R34.2
- new net: Q24.1 (C), R24.1
- new net: D3.2 (A), R61.2
- new net: Q32.2 (B), R31.2
- new net: D1.1 (K), D10.1 (K), D11.1 (K), D12.1 (K), D13.1 (K), D14.1 (K), D2.1 (K), D3.1 (K), D4.1 (K), D5.1 (K), D6.1 (K), D7.1 (K), D8.1 (K), D9.1 (K), Q32.3 (C)
- new net: Q1.1 (C), R1.1
- new net: Q1.2 (B), R32.2
- new net: Q3.1 (C), R3.1
- new net: D6.2 (A), R64.2
- new net: Q32.2 (B), R28.2
- new net: Q6.1 (C), R6.1
- new net: Q2.1 (C), R2.1
- new net: Q12.1 (C), R12.1
- new net: Q12.2 (B), R43.2
- new net: Q32.2 (B), R57.2
- new net: Q5.1 (C), R5.1
- new net: D12.2 (A), R70.2
- new net: Q32.2 (B), R30.2
- new net: D11.2 (A), R69.2
- new net: D14.2 (A), R72.2
- new net: D10.2 (A), R68.2
- new net: Q13.2 (B), R44.2
- new net: D1.2 (A), R59.2
- new net: Q8.1 (C), R8.1
- new net: D4.2 (A), R62.2
- new net: Q8.2 (B), R39.2
- new net: Q32.2 (B), R26.2
- new net: Q32.2 (B), R58.2
- new net: Q5.2 (B), R36.2
- new net: Q18.1 (C), R18.1
- new net: Q18.2 (B), R49.2
- new net: D7.2 (A), R65.2
- new net: Q32.2 (B), R27.2
- new net: Q4.1 (C), R4.1
- new net: Q10.1 (C), R10.1
- new net: Q10.2 (B), R41.2
- new net: Q32.2 (B), R29.2
- new net: Q7.1 (C), R7.1
- new net: Q7.2 (B), R38.2
- new net: Q14.2 (B), R45.2
- new net: Q32.2 (B), R25.2
- new net: Q14.1 (C), R14.1
- new net: Q15.1 (C), R15.1
- new net: D2.2 (A), R60.2
- new net: Q21.1 (C), R21.1
- new net: Q22.1 (C), R22.1
- new net: Q22.2 (B), R53.2
- new net: Q6.2 (B), R37.2
- new net: Q11.2 (B), R42.2
- new net: Q9.2 (B), R40.2
- new net: Q19.1 (C), R19.1
- new net: Q19.2 (B), R50.2
- new net: Q21.2 (B), R52.2
- new net: Q24.2 (B), R55.2
- new net: D8.2 (A), R66.2
- new net: Q2.2 (B), R33.2
- new net: Q23.1 (C), R23.1
- new net: Q23.2 (B), R54.2
- new net: Q11.1 (C), R11.1
- new net: Q13.1 (C), R13.1
- new net: D13.2 (A), R71.2
- new net: Q9.1 (C), R9.1
- new net: Q15.2 (B), R46.2
- new net: Q20.1 (C), R20.1
- new net: Q4.2 (B), R35.2
- new net: D5.2 (A), R63.2
- new net: D9.2 (A), R67.2
- new net: Q20.2 (B), R51.2
- new net +12V: C66.1, C67.1, R107.2
- new net +5V: C1.1, C2.1, R1.2, R10.2, R11.2, R12.2, R13.2, R14.2, R15.2, R16.2, R17.2, R18.2, R19.2, R2.2, R20.2, R21.2, R22.2, R23.2, R24.2, R3.2, R4.2, R5.2, R59.1, R6.2, R60.1, R61.1, R62.1, R63.1, R64.1, R65.1, R66.1, R67.1, R68.1, R69.1, R7.2, R70.1, R71.1, R72.1, R8.2, R9.2
- new net BACKLIGHT_CONTROL: R57.1, R58.1
- new net LEDS_ANODE_0: Q1.3 (E)
- new net LEDS_ANODE_1: Q2.3 (E)
- new net LEDS_ANODE_10: Q11.3 (E)
- new net LEDS_ANODE_11: Q12.3 (E)
- new net LEDS_ANODE_12: Q13.3 (E)
- new net LEDS_ANODE_13: Q14.3 (E)
- new net LEDS_ANODE_14: Q15.3 (E)
- new net LEDS_ANODE_15: Q16.3 (E)
- new net LEDS_ANODE_16: Q17.3 (E)
- new net LEDS_ANODE_17: Q18.3 (E)
- new net LEDS_ANODE_18: Q19.3 (E)
- new net LEDS_ANODE_19: Q20.3 (E)
- new net LEDS_ANODE_2: Q3.3 (E)
- new net LEDS_ANODE_20: Q21.3 (E)
- new net LEDS_ANODE_21: Q22.3 (E)
- new net LEDS_ANODE_22: Q23.3 (E)
- new net LEDS_ANODE_23: Q24.3 (E)
- new net LEDS_ANODE_3: Q4.3 (E)
- new net LEDS_ANODE_4: Q5.3 (E)
- new net LEDS_ANODE_5: Q6.3 (E)
- new net LEDS_ANODE_6: Q7.3 (E)
- new net LEDS_ANODE_7: Q8.3 (E)
- new net LEDS_ANODE_8: Q9.3 (E)
- new net LEDS_ANODE_9: Q10.3 (E)
- new net LEDS_SEGMENTS_ROW_A: Q32.3 (C)
- new net LEDS_SEGMENTS_ROW_B: Q32.3 (C)
- new net LEDS_SEGMENTS_ROW_C: Q32.3 (C)
- new net LEDS_SEGMENTS_ROW_D: Q32.3 (C)
- new net LEDS_SEGMENTS_ROW_E: Q32.3 (C)
- new net LEDS_SEGMENTS_ROW_F: Q32.3 (C)
- new net LEDS_SEGMENTS_ROW_G: Q32.3 (C)
- new net LED_MULTIPLEX_0: R32.1
- new net LED_MULTIPLEX_1: R33.1
- new net LED_MULTIPLEX_10: R42.1
- new net LED_MULTIPLEX_11: R43.1
- new net LED_MULTIPLEX_12: R44.1
- new net LED_MULTIPLEX_13: R45.1
- new net LED_MULTIPLEX_14: R46.1
- new net LED_MULTIPLEX_15: R47.1
- new net LED_MULTIPLEX_16: R48.1
- new net LED_MULTIPLEX_17: R49.1
- new net LED_MULTIPLEX_18: R50.1
- new net LED_MULTIPLEX_19: R51.1
- new net LED_MULTIPLEX_2: R34.1
- new net LED_MULTIPLEX_20: R52.1
- new net LED_MULTIPLEX_21: R53.1
- new net LED_MULTIPLEX_22: R54.1
- new net LED_MULTIPLEX_23: R55.1
- new net LED_MULTIPLEX_3: R35.1
- new net LED_MULTIPLEX_4: R36.1
- new net LED_MULTIPLEX_5: R37.1
- new net LED_MULTIPLEX_6: R38.1
- new net LED_MULTIPLEX_7: R39.1
- new net LED_MULTIPLEX_8: R40.1
- new net LED_MULTIPLEX_9: R41.1
- new net LED_MULTIPLEX_A: R25.1
- new net LED_MULTIPLEX_B: R26.1
- new net LED_MULTIPLEX_C: R27.1
- new net LED_MULTIPLEX_D: R28.1
- new net LED_MULTIPLEX_E: R29.1
- new net LED_MULTIPLEX_F: R30.1
- new net LED_MULTIPLEX_G: R31.1
- new net NRST: J17.4 (Pin_4)
- new net SWCLK: J17.3 (Pin_3)
- new net SWDIO: J17.2 (Pin_2)
Other:
- note added: "12V filament bulbs, 80mA each"
- note added: "brightness is PWM controlled"
- note added: "check this module can actually handle the current of the number of leds being used"
- note added: "including button backlight"
- note added: "use this to adjust max brightness"
- note removed: "backlight and a/t arm toggle reset"
