File: cockpit/panels/MCP/hardware/electronics/mcpElectronics/heading.kicad_sch (KiCad schematic)
At the start: 26 parts

Commit message: update
Parts:
- removed C? (x3): 100n, symbol Device:C
- removed R? (x3): 1k, symbol Device:R
- removed RV?: 4k7, symbol Device:R_Potentiometer
- removed U? (x3): TLC5916IDR, TLC5916IDR:SOIC127P600X175-16N, symbol TLC5916IDR:TLC5916IDR
- removed U? (x3): WHITE_7_SEGMENT_LED, Display_7Segment:Sx39-1xxxxx, symbol Display_Character:SA39-11EWA
- added C4 (x3): 100n, Capacitor_SMD:C_0402_1005Metric, symbol Device:C
- added J16: Bank Angle Selector, Connector_PinHeader_2.54mm:PinHeader_1x06_P2.54mm_Vertical, symbol Connector:Conn_01x06_Pin
- added J18 (x3): WHITE_7_SEGMENT_LED, Connector_PinHeader_2.54mm:PinHeader_1x09_P2.54mm_Vertical, symbol Connector:Conn_01x09_Pin
- added R131, R135: 10k, Resistor_SMD:R_0402_1005Metric, symbol Device:R
- added R132: 1k, Resistor_SMD:R_0402_1005Metric, symbol Device:R
- added R133: 2k2, Resistor_SMD:R_0402_1005Metric, symbol Device:R
- added R134: 5k6, Resistor_SMD:R_0402_1005Metric, symbol Device:R
- added R136: 22k, Resistor_SMD:R_0402_1005Metric, symbol Device:R
- added R138 (x2): 4k7, Resistor_SMD:R_0402_1005Metric, symbol Device:R
- C55, C56, C57, C58: renamed from C?; footprint (none) -> Capacitor_SMD:C_0402_1005Metric
- R118, R119, R120, R121: renamed from R?; footprint (none) -> Resistor_SMD:R_0402_1005Metric
- SW12, SW13, SW14, SW16: renamed from SW?; footprint (none) -> Button_Switch_THT:SW_PUSH_6mm_H5mm
- SW15: renamed from SW?; footprint (none) -> Rotary_Encoder:RotaryEncoder_Bourns_Vertical_PEC12R-3x17F-Nxxxx
Connections:
- net +3V3: now also J16.6 (Pin_6), R138.1, R138.1
- net BANK_ANGLE_SELECT: now also R131.1, R132.1, R133.1, R134.1, R135.1, R136.1
- net Earth: now also C4.2, C4.2, C4.2, R131.2
- net HEADING_DEC: now also R138.2
- net HEADING_INC: now also R138.2
- new net: J16.4 (Pin_4), R133.2
- new net: J16.3 (Pin_3), R134.2
- new net: J16.5 (Pin_5), R132.2
- new net: J16.1 (Pin_1), R136.2
- new net: J16.2 (Pin_2), R135.2
- new net LEDS_ANODE_10: C4.1, J18.8 (Pin_8), J18.9 (Pin_9)
- new net LEDS_ANODE_11: C4.1, J18.8 (Pin_8), J18.9 (Pin_9)
- new net LEDS_ANODE_9: C4.1, J18.8 (Pin_8), J18.9 (Pin_9)
- new net LEDS_SEGMENTS_ROW_A: J18.1 (Pin_1), J18.1 (Pin_1), J18.1 (Pin_1)
- new net LEDS_SEGMENTS_ROW_B: J18.2 (Pin_2), J18.2 (Pin_2), J18.2 (Pin_2)
- new net LEDS_SEGMENTS_ROW_C: J18.3 (Pin_3), J18.3 (Pin_3), J18.3 (Pin_3)
- new net LEDS_SEGMENTS_ROW_D: J18.4 (Pin_4), J18.4 (Pin_4), J18.4 (Pin_4)
- new net LEDS_SEGMENTS_ROW_E: J18.5 (Pin_5), J18.5 (Pin_5), J18.5 (Pin_5)
- new net LEDS_SEGMENTS_ROW_F: J18.6 (Pin_6), J18.6 (Pin_6), J18.6 (Pin_6)
- new net LEDS_SEGMENTS_ROW_G: J18.7 (Pin_7), J18.7 (Pin_7), J18.7 (Pin_7)
- no-connect marks 7 -> 0
