File: cockpit/panels/MCP/hardware/electronics/mcpElectronics/iasmach.kicad_sch (KiCad schematic)
At the start: 36 parts

Commit message: update
Parts:
- removed C? (x4): 100n, symbol Device:C
- removed R? (x3): 1k, symbol Device:R
- removed R?: 10k, symbol Device:R
- removed U?: TLC5926IDWR, symbol TLC5916IDR:TLC5926IDWR
- removed U? (x3): WHITE_7_SEGMENT_LED, Display_7Segment:Sx39-1xxxxx, symbol Display_Character:SA39-11EWA
- removed U? (x3): TLC5916IDR, TLC5916IDR:SOIC127P600X175-16N, symbol TLC5916IDR:TLC5916IDR
- added C3, C4, C5, C6, C7: 100n, Capacitor_SMD:C_0402_1005Metric, symbol Device:C
- added J18 (x3): WHITE_7_SEGMENT_LED, Connector_PinHeader_2.54mm:PinHeader_1x09_P2.54mm_Vertical, symbol Connector:Conn_01x09_Pin
- added J2: A/T_TOGGLE_RESET_ELECTROMAGNET, Connector_PinHeader_2.54mm:PinHeader_1x02_P2.54mm_Vertical, symbol Connector_Generic:Conn_01x02
- added J3: WHITE_ALPHANUMERIC_LED, Connector_PinHeader_2.54mm:PinHeader_1x14_P2.54mm_Vertical, symbol Connector_Generic:Conn_01x14
- added Q32: S8050, Package_TO_SOT_THT:TO-92_Inline, symbol Transistor_BJT:S8050
- added R138, R139: 4k7, Resistor_SMD:R_0402_1005Metric, symbol Device:R
- added R25: 560R, Resistor_SMD:R_0402_1005Metric, symbol Device:R
- C49, C50, C51, C52, C53, C54: renamed from C?; footprint (none) -> Capacitor_SMD:C_0402_1005Metric
- R111, R112, R113, R114, R115, R116, R117: renamed from R?; footprint (none) -> Resistor_SMD:R_0402_1005Metric
- SW10, SW4, SW5, SW7, SW8, SW9: renamed from SW?; footprint (none) -> Button_Switch_THT:SW_PUSH_6mm_H5mm
- SW11: renamed from SW?; footprint (none) -> Connector_PinHeader_2.54mm:PinHeader_1x02_P2.54mm_Vertical
- SW6: renamed from SW?; footprint (none) -> Rotary_Encoder:RotaryEncoder_Bourns_Vertical_PEC12R-3x17F-Nxxxx
Connections:
- net +3V3: now also R138.1, R139.1
- net Earth: now also C3.2, C4.2, C5.2, C6.2, C7.2, Q32.1 (E)
- net IASMACH_DEC: now also R139.2
- net IASMACH_INC: now also R138.2
- net A/T_ARM_OFF: no longer names the net of SW11.3 (C)
- new net: J2.1 (Pin_1), Q32.3 (C)
- new net: Q32.2 (B), R25.2
- new net +12V: J2.2 (Pin_2)
- new net A/T_TOGGLE_RESET: R25.1
- new net LEDS_ANODE_0: C3.1, J18.8 (Pin_8), J18.9 (Pin_9)
- new net LEDS_ANODE_1: C4.1, J18.8 (Pin_8), J18.9 (Pin_9)
- new net LEDS_ANODE_2: C5.1, J18.8 (Pin_8), J18.9 (Pin_9)
- new net LEDS_ANODE_22: C7.1, J3.13 (Pin_13)
- new net LEDS_ANODE_23: C6.1, J3.14 (Pin_14)
- new net LEDS_SEGMENTS_ROW_A: J18.1 (Pin_1), J18.1 (Pin_1), J18.1 (Pin_1), J3.1 (Pin_1), J3.8 (Pin_8)
- new net LEDS_SEGMENTS_ROW_B: J18.2 (Pin_2), J18.2 (Pin_2), J18.2 (Pin_2), J3.2 (Pin_2), J3.9 (Pin_9)
- new net LEDS_SEGMENTS_ROW_C: J18.3 (Pin_3), J18.3 (Pin_3), J18.3 (Pin_3), J3.10 (Pin_10), J3.3 (Pin_3)
- new net LEDS_SEGMENTS_ROW_D: J18.4 (Pin_4), J18.4 (Pin_4), J18.4 (Pin_4), J3.11 (Pin_11), J3.4 (Pin_4)
- new net LEDS_SEGMENTS_ROW_E: J18.5 (Pin_5), J18.5 (Pin_5), J18.5 (Pin_5), J3.12 (Pin_12), J3.5 (Pin_5)
- new net LEDS_SEGMENTS_ROW_F: J18.6 (Pin_6), J18.6 (Pin_6), J18.6 (Pin_6), J3.6 (Pin_6)
- new net LEDS_SEGMENTS_ROW_G: J18.7 (Pin_7), J18.7 (Pin_7), J18.7 (Pin_7), J3.7 (Pin_7)
- no-connect marks 5 -> 1
Other:
- note added: "14 connections required (including 2x CA)"
- note added: "DOT REQUIRED"
- note added: "M, B, A characters required"
- note removed: "CHECK THAT DIFFERENT LED DRIVERS USING DIFFERENT NUMBERS OF PINOUTS CAN BE USED TOGETHER"
