File: cockpit/panels/MCP/hardware/electronics/mcpElectronics/indication_lights.kicad_sch (KiCad schematic)
At the start: 43 parts

Commit message: update schematic
Connections:
- net SPEED_ARM_IND: now reaches D?.1 (K), U?.10 (~{OUT5})
- net MA_PRI_IND: now reaches D?.1 (K), U?.12 (~{OUT7})
- net LNAV_IND: now reaches D?.1 (K), U?.6 (~{OUT1})
- net V/S_IND: now reaches D?.1 (K), U?.7 (~{OUT2})
- net CMD_A_IND: now reaches D?.1 (K), U?.8 (~{OUT3})
- net VNAV_IND: now reaches D?.1 (K), U?.9 (~{OUT4})
- net LVL_CHG_IND: now reaches D?.1 (K), U?.8 (~{OUT3})
- net MA_SEC_IND: now reaches D?.1 (K), U?.5 (~{OUT0})
- net N1_ARM_IND: now reaches D?.1 (K), U?.11 (~{OUT6})
- net CWS_B_IND: now reaches D?.1 (K), U?.11 (~{OUT6})
- net A/T_ARM_IND: now reaches D?.1 (K), U?.12 (~{OUT7})
- net VOR_LOC_IND: now reaches D?.1 (K), U?.5 (~{OUT0})
- net HDG_SEL_IND: now reaches D?.1 (K), U?.7 (~{OUT2})
- net ALT_HLD_IND: now reaches D?.1 (K), U?.6 (~{OUT1})
- net CMD_B_IND: now reaches D?.1 (K), U?.9 (~{OUT4})
- net CWS_A_IND: now reaches D?.1 (K), U?.10 (~{OUT5})
- net APP_IND: now reaches D?.1 (K), U?.5 (~{OUT0})
Changed lines of the file:
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@@
     (stroke (width 0) (type default) (color 0 0 0 0))
+  )
+  (label "SPEED_ARM_IND" (at 82.55 40.64 0)
+    (effects (font (size 1.27 1.27)) (justify left bottom))
+  )
+  (label "VNAV_IND" (at 82.55 38.1 0)
+    (effects (font (size 1.27 1.27)) (justify left bottom))
+  )
+  (label "VOR_LOC_IND" (at 82.55 27.94 0)
+    (effects (font (size 1.27 1.27)) (justify left bottom))
+  )
+  (label "A{slash}T_ARM_IND" (at 82.55 45.72 0)
+    (effects (font (size 1.27 1.27)) (justify left bottom))
+  )
+  (label "N1_ARM_IND" (at 82.55 43.18 0)
+    (effects (font (size 1.27 1.27)) (justify left bottom))
+  )
+  (label "LVL_CHG_IND" (at 82.55 35.56 0)
+    (effects (font (size 1.27 1.27)) (justify left bottom))
+  )
+  (label "V{slash}S_IND" (at 82.55 92.71 0)
+    (effects (font (size 1.27 1.27)) (justify left bottom))
+  )
+  (label "CWS_A_IND" (at 82.55 100.33 0)
+    (effects (font (size 1.27 1.27)) (justify left bottom))
+  )
+  (label "MA_SEC_IND" (at 82.55 147.32 0)
+    (effects (font (size 1.27 1.27)) (justify left bottom))
+  )
+  (label "CMD_B_IND" (at 82.55 97.79 0)
+    (effects (font (size 1.27 1.27)) (justify left bottom))
+  )
+  (label "CMD_A_IND" (at 82.55 95.25 0)
+    (effects (font (size 1.27 1.27)) (justify left bottom))
+  )
+  (label "ALT_HLD_IND" (at 82.55 90.17 0)
+    (effects (font (size 1.27 1.27)) (justify left bottom))
+  )
+  (label "MA_PRI_IND" (at 82.55 105.41 0)
+    (effects (font (size 1.27 1.27)) (justify left bottom))
+  )
+  (label "APP_IND" (at 82.55 87.63 0)
+    (effects (font (size 1.27 1.27)) (justify left bottom))
+  )
+  (label "HDG_SEL_IND" (at 82.55 33.02 0)
+    (effects (font (size 1.27 1.27)) (justify left bottom))
+  )
+  (label "LNAV_IND" (at 82.55 30.48 0)
+    (effects (font (size 1.27 1.27)) (justify left bottom))
+  )
+  (label "CWS_B_IND" (at 82.55 102.87 0)
+    (effects (font (size 1.27 1.27)) (justify left bottom))
   )
   (global_label "INDICATION_OE" (shape input) (at 46.99 147.32 180) (fields_autoplaced)

Commit message: update
Parts:
- removed C? (x3): 100n, symbol Device:C
- removed D? (x17): LED, symbol Device:LED
- removed R? (x17): 330R, symbol Device:R
- removed R? (x3): 1k, symbol Device:R
- removed U? (x3): TLC5916IDR, TLC5916IDR:SOIC127P600X175-16N, symbol TLC5916IDR:TLC5916IDR
- added D15, D16, D17, D18, D19, D20, D21, D22, D23, D24, D25, D26, D27, D28, D29, D30, D31: LED, Connector_PinHeader_2.54mm:PinHeader_1x02_P2.54mm_Vertical, symbol Device:LED
- added Q8 (x17): C945, Package_TO_SOT_THT:TO-92_Inline, symbol Simulation_SPICE:NPN
- added R39 (x17), R8 (x17): 560R, Resistor_SMD:R_0402_1005Metric, symbol Device:R
Connections:
- net ALT_HLD_IND: now also R39.1
- net APP_IND: now also R39.1
- net A/T_ARM_IND: now also R39.1
- net CMD_A_IND: now also R39.1
- net CMD_B_IND: now also R39.1
- net CWS_A_IND: now also R39.1
- net CWS_B_IND: now also R39.1
- net Earth: now also Q8.3 (E), Q8.3 (E), Q8.3 (E), Q8.3 (E), Q8.3 (E), Q8.3 (E), Q8.3 (E), Q8.3 (E), Q8.3 (E), Q8.3 (E), Q8.3 (E), Q8.3 (E), Q8.3 (E), Q8.3 (E), Q8.3 (E), Q8.3 (E), Q8.3 (E)
- net HDG_SEL_IND: now also R39.1
- net LNAV_IND: now also R39.1
- net LVL_CHG_IND: now also R39.1
- net MA_PRI_IND: now also R39.1
- net MA_SEC_IND: now also R39.1
- net N1_ARM_IND: now also R39.1
- net SPEED_ARM_IND: now also R39.1
- net VNAV_IND: now also R39.1
- net VOR_LOC_IND: now also R39.1
- net V/S_IND: now also R39.1
- new net: D22.1 (K), R8.2
- new net: Q8.1 (C), R8.1 (x17)
- new net: D25.1 (K), R8.2
- new net: D31.1 (K), R8.2
- new net: Q8.2 (B), R39.2 (x17)
- new net: D29.1 (K), R8.2
- new net: D23.1 (K), R8.2
- new net: D27.1 (K), R8.2
- new net: D30.1 (K), R8.2
- new net: D15.1 (K), R8.2
- new net: D21.1 (K), R8.2
- new net: D28.1 (K), R8.2
- new net: D17.1 (K), R8.2
- new net: D18.1 (K), R8.2
- new net: D19.1 (K), R8.2
- new net: D24.1 (K), R8.2
- new net: D26.1 (K), R8.2
- new net: D16.1 (K), R8.2
- new net: D20.1 (K), R8.2
- new net +5V: D15.2 (A), D16.2 (A), D17.2 (A), D18.2 (A), D19.2 (A), D20.2 (A), D21.2 (A), D22.2 (A), D23.2 (A), D24.2 (A), D25.2 (A), D26.2 (A), D27.2 (A), D28.2 (A), D29.2 (A), D30.2 (A), D31.2 (A)
- no-connect marks 8 -> 0
